File: interruptor.sch (KiCad schematic (older format))
At the start: 23 parts, among them J1 220v, J2 tx/rx, J3 Screw_Terminal_01x03, J4 Screw_Terminal_01x03, J5 Int_1, J6 int_2, J7 switch, K1 SRD-05VDC-SL-C, K2 SRD-05VDC-SL-C, Q1 PN2222A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

Commit message: colocacion componentes en pcb y conexionado
Connections:
- no-connect marks 5 -> 6
Changed lines of the file:
@@
 	1    0    0    -1
 $EndComp
+Text GLabel 5750 5350 0    50   Input ~ 0
+Relay_1
 Text GLabel 5750 5250 0    50   Input ~ 0
-Relay_1
-Text GLabel 5750 5350 0    50   Input ~ 0
 Relay_2
 Text GLabel 4300 4150 3    50   Input ~ 0
@@
 Wire Wire Line
 	5650 5450 5900 5450
+NoConn ~ 8050 5100
 $EndSCHEMATC

Commit message: pistas dibujadas
Changed lines of the file:
@@
 	1    0    0    -1
 $EndComp
-Text GLabel 5750 5350 0    50   Input ~ 0
+Text GLabel 5750 5250 0    50   Input ~ 0
 Relay_1
-Text GLabel 5750 5250 0    50   Input ~ 0
+Text GLabel 5500 5150 0    50   Input ~ 0
 Relay_2
 Text GLabel 4300 4150 3    50   Input ~ 0
@@
 Wire Wire Line
 	5800 2450 5800 2800
-Text GLabel 5500 5150 0    50   Input ~ 0
+Text GLabel 5750 5350 0    50   Input ~ 0
 int_1
 Connection ~ 6800 6050
