File: interruptorRev2.kicad_pcb (KiCad board)
At the start: 2 copper layers, 43 x 47 mm, 20 parts, among them J1 220v, J2 tx/rx, J3 Screw_Terminal_01x03, J4 Screw_Terminal_01x03, J5 Int_1, J6 int_2, J7 switch, Q1 PN2222A, Q2 PN2222A, U1 HLK-PM01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

Commit message: pines para flashear
Parts:
- J2: value tx/rx -> Conn_01x04; footprint Connector_PinHeader_2.54mm:PinHeader_1x03_P2.54mm_Vertical -> Connector_PinHeader_2.54mm:PinHeader_1x04_P2.54mm_Vertical
- J7: value switch -> Conn_01x02; footprint Connector_PinHeader_2.54mm:PinHeader_1x03_P2.54mm_Vertical -> Connector_PinHeader_2.54mm:PinHeader_1x02_P2.54mm_Vertical
- moved J7 3.29 mm to (107.8, 106.6)
- moved J2 0.92 mm to (121.3, 106.5)
Connections:
- J2 pad 1: Net-(J2-Pad1) -> vcc
- J2 pad 2: Net-(J2-Pad2) -> GND
- J2 pad 3: GND -> Net-(J2-Pad3)
- J7 pad 1: (no net) -> Net-(J7-Pad1)
- J7 pad 2: Net-(J7-Pad2) -> GND
- R3 pad 1: Net-(J2-Pad2) -> Net-(J2-Pad4)
- U3 pad 12: Net-(J7-Pad2) -> Net-(J7-Pad1)
- U3 pad 16: Net-(J2-Pad1) -> Net-(J2-Pad3)
