File: file5D5B915D.sch (KiCad schematic (older format))
At the start: 22 parts, among them Q3 2N7002, U2 HLW8012

Commit message: esquema dividido por secciones
Parts:
- C1, C2, C3, C4, C5: footprint (none) -> Capacitor_SMD:C_0805_2012Metric
- R10, R11, R12, R13, R14, R15, R16, R17, R18, R19, R20, R6, R7, R8: footprint (none) -> Resistor_SMD:R_0805_2012Metric_Pad1.15x1.40mm_HandSolder
- R9: footprint (none) -> espurna-h:2512
- U2: footprint (none) -> espurna-h:SOP8
Connections:
- wire segments 69 -> 68
Changed lines of the file:
@@
 F 0 "U2" H 6000 3286 59  0000 C CNN
 F 1 "HLW8012" H 6000 3181 59  0000 C CNN
-F 2 "" H 6000 2800 50  0001 C CNN
+F 2 "espurna-h:SOP8" H 6000 2800 50  0001 C CNN
 F 3 "" H 6000 2800 50  0001 C CNN
 	1    6000 2800
@@
 F 0 "R9" V 3493 2300 50  0000 C CNN
 F 1 "0.001R" V 3584 2300 50  0000 C CNN
-F 2 "" V 3630 2300 50  0001 C CNN
+F 2 "espurna-h:2512" V 3630 2300 50  0001 C CNN
 F 3 "~" H 3700 2300 50  0001 C CNN
 	1    3700 2300
@@
 F 0 "R8" H 3470 2596 50  0000 L CNN
 F 1 "1K" H 3470 2505 50  0000 L CNN
-F 2 "" V 3330 2550 50  0001 C CNN
+F 2 "Resistor_SMD:R_0805_2012Metric_Pad1.15x1.40mm_HandSolder" V 3330 2550 50  0001 C CNN
 F 3 "~" H 3400 2550 50  0001 C CNN
 	1    3400 2550
@@
 F 0 "R11" V 4050 2550 50  0000 L CNN
 F 1 "1K" H 4020 2505 50  0000 L CNN
-F 2 "" V 3880 2550 50  0001 C CNN
+F 2 "Resistor_SMD:R_0805_2012Metric_Pad1.15x1.40mm_HandSolder" V 3880 2550 50  0001 C CNN
 F 3 "~" H 3950 2550 50  0001 C CNN
 	1    3950 2550
@@
 F 0 "R13" V 4300 2550 50  0000 L CNN
 F 1 "0R" H 4270 2505 50  0000 L CNN
-F 2 "" V 4130 2550 50  0001 C CNN
+F 2 "Resistor_SMD:R_0805_2012Metric_Pad1.15x1.40mm_HandSolder" V 4130 2550 50  0001 C CNN
 F 3 "~" H 4200 2550 50  0001 C CNN
 	1    4200 2550
@@
 F 0 "C1" H 3450 3250 50  0000 L CNN
 F 1 "33nF" H 3200 3450 50  0000 L CNN
-F 2 "" H 3438 3200 50  0001 C CNN
+F 2 "Capacitor_SMD:C_0805_2012Metric" H 3438 3200 50  0001 C CNN
 F 3 "~" H 3400 3350 50  0001 C CNN
 	1    3400 3350
@@
 F 0 "C2" H 4000 3250 50  0000 L CNN
 F 1 "33nF" H 3750 3450 50  0000 L CNN
-F 2 "" H 3988 3200 50  0001 C CNN
+F 2 "Capacitor_SMD:C_0805_2012Metric" H 3988 3200 50  0001 C CNN
 F 3 "~" H 3950 3350 50  0001 C CNN
 	1    3950 3350
@@
 F 0 "C3" H 4600 3250 50  0000 L CNN
 F 1 "100nF" H 4300 3450 50  0000 L CNN
-F 2 "" H 4588 3200 50  0001 C CNN
+F 2 "Capacitor_SMD:C_0805_2012Metric" H 4588 3200 50  0001 C CNN
 F 3 "~" H 4550 3350 50  0001 C CNN
 	1    4550 3350
@@
 F 0 "C4" H 4950 3250 50  0000 L CNN
 F 1 "1uF" H 4750 3450 50  0000 L CNN
-F 2 "" H 4938 3200 50  0001 C CNN
+F 2 "Capacitor_SMD:C_0805_2012Metric" H 4938 3200 50  0001 C CNN
 F 3 "~" H 4900 3350 50  0001 C CNN
 	1    4900 3350
@@
 F 0 "C5" H 5350 3250 50  0000 L CNN
 F 1 "100nF" H 5050 3450 50  0000 L CNN
-F 2 "" H 5338 3200 50  0001 C CNN
+F 2 "Capacitor_SMD:C_0805_2012Metric" H 5338 3200 50  0001 C CNN
 F 3 "~" H 5300 3350 50  0001 C CNN
 	1    5300 3350
@@
 F 0 "R16" V 6750 2800 50  0000 C CNN
 F 1 "10K" V 6850 2800 50  0000 C CNN
-F 2 "" V 6780 2800 50  0001 C CNN
+F 2 "Resistor_SMD:R_0805_2012Metric_Pad1.15x1.40mm_HandSolder" V 6780 2800 50  0001 C CNN
 F 3 "~" H 6850 2800 50  0001 C CNN
 	1    6850 2800
@@
 F 0 "R17" V 6750 3000 50  0000 C CNN
 F 1 "10K" V 6850 3000 50  0000 C CNN
-F 2 "" V 6780 3000 50  0001 C CNN
+F 2 "Resistor_SMD:R_0805_2012Metric_Pad1.15x1.40mm_HandSolder" V 6780 3000 50  0001 C CNN
 F 3 "~" H 6850 3000 50  0001 C CNN
 	1    6850 3000
@@
 F 0 "R18" H 7120 3396 50  0000 L CNN
 F 1 "15K" H 7120 3305 50  0000 L CNN
-F 2 "" V 6980 3350 50  0001 C CNN
+F 2 "Resistor_SMD:R_0805_2012Metric_Pad1.15x1.40mm_HandSolder" V 6980 3350 50  0001 C CNN
 F 3 "~" H 7050 3350 50  0001 C CNN
 	1    7050 3350
@@
 F 0 "R19" H 7470 3396 50  0000 L CNN
 F 1 "15K" H 7470 3305 50  0000 L CNN
-F 2 "" V 7330 3350 50  0001 C CNN
+F 2 "Resistor_SMD:R_0805_2012Metric_Pad1.15x1.40mm_HandSolder" V 7330 3350 50  0001 C CNN
 F 3 "~" H 7400 3350 50  0001 C CNN
 	1    7400 3350
@@
 F 0 "R20" H 8420 2396 50  0000 L CNN
 F 1 "10K" H 8420 2305 50  0000 L CNN
-F 2 "" V 8280 2350 50  0001 C CNN
+F 2 "Resistor_SMD:R_0805_2012Metric_Pad1.15x1.40mm_HandSolder" V 8280 2350 50  0001 C CNN
 F 3 "~" H 8350 2350 50  0001 C CNN
 	1    8350 2350
@@
 	4900 3500 5300 3500
 Connection ~ 4900 3500
-Text Label 3050 2300 0    50   ~ 0
-LINE_I
-Text Label 4300 2300 0    50   ~ 0
-LINE_L
 Wire Wire Line
 	3950 2700 3950 3000
@@
 F 0 "R6" H 2970 5196 50  0000 L CNN
 F 1 "470k" H 2970 5105 50  0000 L CNN
-F 2 "" V 2830 5150 50  0001 C CNN
+F 2 "Resistor_SMD:R_0805_2012Metric_Pad1.15x1.40mm_HandSolder" V 2830 5150 50  0001 C CNN
 F 3 "~" H 2900 5150 50  0001 C CNN
 	1    2900 5150
@@
 F 0 "R7" H 3370 5196 50  0000 L CNN
 F 1 "470k" H 3370 5105 50  0000 L CNN
-F 2 "" V 3230 5150 50  0001 C CNN
+F 2 "Resistor_SMD:R_0805_2012Metric_Pad1.15x1.40mm_HandSolder" V 3230 5150 50  0001 C CNN
 F 3 "~" H 3300 5150 50  0001 C CNN
 	1    3300 5150
@@
 F 0 "R10" H 3770 5196 50  0000 L CNN
 F 1 "470k" H 3770 5105 50  0000 L CNN
-F 2 "" V 3630 5150 50  0001 C CNN
+F 2 "Resistor_SMD:R_0805_2012Metric_Pad1.15x1.40mm_HandSolder" V 3630 5150 50  0001 C CNN
 F 3 "~" H 3700 5150 50  0001 C CNN
 	1    3700 5150
@@
 F 0 "R12" H 4170 5196 50  0000 L CNN
 F 1 "470k" H 4170 5105 50  0000 L CNN
-F 2 "" V 4030 5150 50  0001 C CNN
+F 2 "Resistor_SMD:R_0805_2012Metric_Pad1.15x1.40mm_HandSolder" V 4030 5150 50  0001 C CNN
 F 3 "~" H 4100 5150 50  0001 C CNN
 	1    4100 5150
@@
 F 0 "R14" H 4570 5196 50  0000 L CNN
 F 1 "470k" H 4570 5105 50  0000 L CNN
-F 2 "" V 4430 5150 50  0001 C CNN
+F 2 "Resistor_SMD:R_0805_2012Metric_Pad1.15x1.40mm_HandSolder" V 4430 5150 50  0001 C CNN
 F 3 "~" H 4500 5150 50  0001 C CNN
 	1    4500 5150
@@
 F 0 "R15" H 5120 5196 50  0000 L CNN
 F 1 "1K" H 5120 5105 50  0000 L CNN
-F 2 "" V 4980 5150 50  0001 C CNN
+F 2 "Resistor_SMD:R_0805_2012Metric_Pad1.15x1.40mm_HandSolder" V 4980 5150 50  0001 C CNN
 F 3 "~" H 5050 5150 50  0001 C CNN
 	1    5050 5150
@@
 Wire Wire Line
 	3200 5000 2900 5000
-Wire Wire Line
-	2900 5300 2900 5550
 Text Label 5100 4600 0    50   ~ 0
 V2P
@@
 	1    0    0    -1
 $EndComp
-Text Label 2900 5550 0    50   ~ 0
-NEUTRAL
 Text GLabel 7650 2800 2    50   Input ~ 0
 GPIO13
@@
 Wire Wire Line
 	4450 2550 4450 2600
+Text GLabel 2900 5300 3    50   Input ~ 0
+NEUTRAL
+Text GLabel 2900 2300 0    50   Input ~ 0
+LINE_I
+Text GLabel 4600 2300 2    50   Input ~ 0
+LINE_L
 $EndSCHEMATC

Commit message: regulador voltaje 3v3
Parts:
- U2: symbol espurna-h-eagle-import:HLW8012 -> interruptorRev2-rescue:HLW8012-espurna-h-eagle-import
Changed lines of the file:
@@
 $EndDescr
 $Comp
-L espurna-h-eagle-import:HLW8012 U2
+L interruptorRev2-rescue:HLW8012-espurna-h-eagle-import U2
 U 1 1 5D5B91CD
 P 6000 2800
+AR Path="/5D5B91CD" Ref="U2"  Part="1"
+AR Path="/5D5B915E/5D5B91CD" Ref="U2"  Part="1"
 F 0 "U2" H 6000 3286 59  0000 C CNN
 F 1 "HLW8012" H 6000 3181 59  0000 C CNN
