File: interruptorRev2.sch (KiCad schematic (older format))
At the start: 23 parts, among them J1 220v, J2 tx/rx, J3 Screw_Terminal_01x03, J4 Screw_Terminal_01x03, J5 Int_1, J6 int_2, J7 switch, K1 SRD-05VDC-SL-C, K2 SRD-05VDC-SL-C, Q1 PN2222A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

Commit message: intentando reducir tamanyo
Parts:
- removed C1, C2: 10uF, Capacitor_SMD:C_1206_3216Metric_Pad1.42x1.75mm_HandSolder, symbol interruptor-rescue:C-device-termostato-rescue
- removed K1: SRD-05VDC-SL-C, SRD-05VDC-SL-C:RELAY_SRD-05VDC-SL-C, symbol SRD-05VDC-SL-C:SRD-05VDC-SL-C
- removed K2: SRD-05VDC-SL-C, RELAY_SRD-05VDC-SL-C, symbol SRD-05VDC-SL-C:SRD-05VDC-SL-C
- removed Q1, Q2: PN2222A, Package_TO_SOT_THT:TO-92_Inline, symbol Transistor_BJT:PN2222A
- removed U2: LM1117-3.3, Package_TO_SOT_SMD:SOT-223, symbol interruptor-rescue:LM1117-3.3-regul-termostato-rescue
- added Q1, Q2: PN2222A, Package_TO_SOT_SMD:SOT-23, symbol pn2222a:PN2222A
- added U4, U5: JRC-21(4100), relays:JRC-21F, symbol reles:JRC-21(4100)
- D1, D2: footprint Diode_THT:D_DO-35_SOD27_P7.62mm_Horizontal -> Diode_SMD:D_1206_3216Metric_Pad1.42x1.75mm_HandSolder
- J1: symbol interruptor-rescue:Conn_01x02_Female-RESCUE-termostato-termostato-rescue -> interruptorRev2-rescue:Conn_01x02_Female-RESCUE-termostato-termostato-rescue-interruptor-rescue
- J2, J5, J6, J7: symbol interruptor-rescue:Conn_01x03_Female-RESCUE-termostato-termostato-rescue -> interruptorRev2-rescue:Conn_01x03_Female-RESCUE-termostato-termostato-rescue-interruptor-rescue
- R1, R2, R3: symbol interruptor-rescue:R-RESCUE-termostato-termostato-rescue -> interruptorRev2-rescue:R-RESCUE-termostato-termostato-rescue-interruptor-rescue
- U1: footprint HLK-PM01 -> HLK-PM01:HLK-PM01
- U3: symbol interruptor-rescue:ESP-07v2-RESCUE-termostato-termostato-rescue -> interruptorRev2-rescue:ESP-07v2-RESCUE-termostato-termostato-rescue-interruptor-rescue
Connections:
- wire segments 86 -> 93

Commit message: pines para flashear
Parts:
- removed J2: tx/rx, Connector_PinHeader_2.54mm:PinHeader_1x03_P2.54mm_Vertical, symbol interruptorRev2-rescue:Conn_01x03_Female-RESCUE-termostato-termostato-rescue-in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
- removed J7: switch, Connector_PinHeader_2.54mm:PinHeader_1x03_P2.54mm_Vertical, symbol interruptorRev2-rescue:Conn_01x03_Female-RESCUE-termostato-termostato-rescue-in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
- added J2: Conn_01x04, Connector_PinHeader_2.54mm:PinHeader_1x04_P2.54mm_Vertical, symbol Connector_Generic:Conn_01x04
- added J7: Conn_01x02, Connector_PinHeader_2.54mm:PinHeader_1x02_P2.54mm_Vertical, symbol Connector_Generic:Conn_01x02
Connections:
- wire segments 93 -> 94
- no-connect marks 6 -> 5
Changed lines of the file:
@@
 	5500 4250 6800 4250
 $Comp
-L interruptorRev2-rescue:Conn_01x03_Female-RESCUE-termostato-termostato-rescue-interruptor-rescue J2
-U 1 1 5A3E9536
-P 7100 3900
-F 0 "J2" H 7100 4100 50  0000 C CNN
-F 1 "tx/rx" H 7100 3700 50  0000 C CNN
-F 2 "Connector_PinHeader_2.54mm:PinHeader_1x03_P2.54mm_Vertical" H 7100 3900 50  0001 C CNN
-F 3 "" H 7100 3900 50  0001 C CNN
-	1    7100 3900
-	0    -1   -1   0
-$EndComp
-$Comp
-L interruptorRev2-rescue:GND-RESCUE-termostato-termostato-rescue-interruptor-rescue #PWR0101
+L interruptorRev2-rescue:GND-RESCUE-termostato-termostato-rescue-interruptor-rescue #PWR?
 U 1 1 5A3E96C3
 P 6800 6250
-F 0 "#PWR0101" H 6800 6000 50  0001 C CNN
+F 0 "#PWR?" H 6800 6000 50  0001 C CNN
 F 1 "GND" H 6800 6100 50  0000 C CNN
 F 2 "" H 6800 6250 50  0001 C CNN
@@
 $EndComp
 $Comp
-L interruptorRev2-rescue:GND-RESCUE-termostato-termostato-rescue-interruptor-rescue #PWR0102
+L interruptorRev2-rescue:GND-RESCUE-termostato-termostato-rescue-interruptor-rescue #PWR?
 U 1 1 5A3E96E1
-P 7200 4150
-F 0 "#PWR0102" H 7200 3900 50  0001 C CNN
-F 1 "GND" H 7200 4000 50  0000 C CNN
-F 2 "" H 7200 4150 50  0001 C CNN
-F 3 "" H 7200 4150 50  0001 C CNN
-	1    7200 4150
+P 6900 4150
+F 0 "#PWR?" H 6900 3900 50  0001 C CNN
+F 1 "GND" H 6900 4000 50  0000 C CNN
+F 2 "" H 6900 4150 50  0001 C CNN
+F 3 "" H 6900 4150 50  0001 C CNN
+	1    6900 4150
 	1    0    0    -1
 $EndComp
@@
 	6800 6050 6800 6250
 $Comp
-L interruptorRev2-rescue:GND-RESCUE-termostato-termostato-rescue-interruptor-rescue #PWR0103
+L interruptorRev2-rescue:GND-RESCUE-termostato-termostato-rescue-interruptor-rescue #PWR?
 U 1 1 5A3E97AE
 P 3750 5300
-F 0 "#PWR0103" H 3750 5050 50  0001 C CNN
+F 0 "#PWR?" H 3750 5050 50  0001 C CNN
 F 1 "GND" H 3750 5150 50  0000 C CNN
 F 2 "" H 3750 5300 50  0001 C CNN
@@
 Connection ~ 3750 4750
 $Comp
-L interruptorRev2-rescue:GND-RESCUE-termostato-termostato-rescue-interruptor-rescue #PWR0109
+L interruptorRev2-rescue:GND-RESCUE-termostato-termostato-rescue-interruptor-rescue #PWR?
 U 1 1 5CD36044
 P 4700 3850
-F 0 "#PWR0109" H 4700 3600 50  0001 C CNN
+F 0 "#PWR?" H 4700 3600 50  0001 C CNN
 F 1 "GND" H 4700 3700 50  0000 C CNN
 F 2 "" H 4700 3850 50  0001 C CNN
@@
 $EndComp
 $Comp
-L interruptorRev2-rescue:GND-RESCUE-termostato-termostato-rescue-interruptor-rescue #PWR0110
+L interruptorRev2-rescue:GND-RESCUE-termostato-termostato-rescue-interruptor-rescue #PWR?
 U 1 1 5CD368F3
 P 6200 3750
-F 0 "#PWR0110" H 6200 3500 50  0001 C CNN
+F 0 "#PWR?" H 6200 3500 50  0001 C CNN
 F 1 "GND" H 6200 3600 50  0000 C CNN
 F 2 "" H 6200 3750 50  0001 C CNN
@@
 	7100 4350 7800 4350
 Wire Wire Line
-	7200 4100 7200 4150
-Wire Wire Line
 	5650 4100 5800 4100
 Wire Wire Line
@@
 	4350 6550 4350 6200
 $Comp
-L interruptorRev2-rescue:GND-RESCUE-termostato-termostato-rescue-interruptor-rescue #PWR01
+L interruptorRev2-rescue:GND-RESCUE-termostato-termostato-rescue-interruptor-rescue #PWR?
 U 1 1 5CDD4154
 P 4450 6300
-F 0 "#PWR01" H 4450 6050 50  0001 C CNN
+F 0 "#PWR?" H 4450 6050 50  0001 C CNN
 F 1 "GND" H 4450 6150 50  0000 C CNN
 F 2 "" H 4450 6300 50  0001 C CNN
@@
 	4250 6350 4250 6200
 $Comp
-L interruptorRev2-rescue:GND-RESCUE-termostato-termostato-rescue-interruptor-rescue #PWR03
+L interruptorRev2-rescue:GND-RESCUE-termostato-termostato-rescue-interruptor-rescue #PWR?
 U 1 1 5CDD4406
 P 9250 5250
-F 0 "#PWR03" H 9250 5000 50  0001 C CNN
+F 0 "#PWR?" H 9250 5000 50  0001 C CNN
 F 1 "GND" H 9250 5100 50  0000 C CNN
 F 2 "" H 9250 5250 50  0001 C CNN
 F 3 "" H 9250 5250 50  0001 C CNN
 	1    9250 5250
-	0    -1   -1   0
-$EndComp
-$Comp
-L interruptorRev2-rescue:Conn_01x03_Female-RESCUE-termostato-termostato-rescue-interruptor-rescue J7
-U 1 1 5CDDC706
-P 9000 4900
-F 0 "J7" H 9000 5100 50  0000 C CNN
-F 1 "switch" H 8900 4700 50  0000 C CNN
-F 2 "Connector_PinHeader_2.54mm:PinHeader_1x03_P2.54mm_Vertical" H 9000 4900 50  0001 C CNN
-F 3 "" H 9000 4900 50  0001 C CNN
-	1    9000 4900
 	0    -1   -1   0
 $EndComp
@@
 	5100 6550 5100 6200
 $Comp
-L interruptorRev2-rescue:GND-RESCUE-termostato-termostato-rescue-interruptor-rescue #PWR02
+L interruptorRev2-rescue:GND-RESCUE-termostato-termostato-rescue-interruptor-rescue #PWR?
 U 1 1 5CDD93E1
 P 5200 6300
-F 0 "#PWR02" H 5200 6050 50  0001 C CNN
+F 0 "#PWR?" H 5200 6050 50  0001 C CNN
 F 1 "GND" H 5200 6150 50  0000 C CNN
 F 2 "" H 5200 6300 50  0001 C CNN
@@
 Wire Wire Line
 	5650 5450 5900 5450
-NoConn ~ 8900 5100
 Wire Wire Line
 	7700 5250 9000 5250
@@
 Text GLabel 3950 4750 2    50   Input ~ 0
 vcc
+$Comp
+L Connector_Generic:Conn_01x04 J2
+U 1 1 5D55AD53
+P 6900 3900
+F 0 "J2" V 6866 3612 50  0000 R CNN
+F 1 "Conn_01x04" V 6775 3612 50  0000 R CNN
+F 2 "Connector_PinHeader_2.54mm:PinHeader_1x04_P2.54mm_Vertical" H 6900 3900 50  0001 C CNN
+F 3 "~" H 6900 3900 50  0001 C CNN
+	1    6900 3900
+	0    -1   -1   0
+$EndComp
+Wire Wire Line
+	6900 4100 6900 4150
+Wire Wire Line
+	6800 4100 6800 4250
+Connection ~ 6800 4250
+$Comp
+L Connector_Generic:Conn_01x02 J7
+U 1 1 5D56056A
+P 9000 4900
+F 0 "J7" V 8966 4712 50  0000 R CNN
+F 1 "Conn_01x02" V 8875 4712 50  0000 R CNN
+F 2 "Connector_PinHeader_2.54mm:PinHeader_1x02_P2.54mm_Vertical" H 9000 4900 50  0001 C CNN
+F 3 "~" H 9000 4900 50  0001 C CNN
+	1    9000 4900
+	0    -1   -1   0
+$EndComp
 $EndSCHEMATC

Commit message: lib rev
Parts:
- Q1, Q2: symbol pn2222a:PN2222A -> interruptorRev2-rescue:PN2222A-pn2222a
- U1: symbol HLK-PM01:HLK-PM01 -> interruptorRev2-rescue:HLK-PM01-HLK-PM01
- U4, U5: symbol reles:JRC-21(4100) -> interruptorRev2-rescue:JRC-21(4100)-reles
Changed lines of the file:
@@
 	5500 4800 5500 5050
 $Comp
-L HLK-PM01:HLK-PM01 U1
+L interruptorRev2-rescue:HLK-PM01-HLK-PM01 U1
 U 1 1 5CD1EF95
 P 3250 4950
@@
 	2500 4750 2750 4750
 $Comp
-L pn2222a:PN2222A Q1
+L interruptorRev2-rescue:PN2222A-pn2222a Q1
 U 1 1 5CEFE5BD
 P 4500 3150
@@
 $EndComp
 $Comp
-L pn2222a:PN2222A Q2
+L interruptorRev2-rescue:PN2222A-pn2222a Q2
 U 1 1 5CEFE632
 P 6000 3150
@@
 NoConn ~ 7700 5050
 $Comp
-L reles:JRC-21(4100) U4
+L interruptorRev2-rescue:JRC-21(4100)-reles U4
 U 1 1 5D07D34E
 P 4100 1550
@@
 Connection ~ 4150 1200
 $Comp
-L reles:JRC-21(4100) U5
+L interruptorRev2-rescue:JRC-21(4100)-reles U5
 U 1 1 5D094505
 P 5550 1600

Commit message: lectura corriente primer esbozo
Parts:
- removed J5: Int_1, Connector_PinHeader_2.54mm:PinHeader_1x03_P2.54mm_Vertical, symbol interruptorRev2-rescue:Conn_01x03_Female-RESCUE-termostato-termostato-rescue-in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
- removed J6: int_2, Connector_PinHeader_2.54mm:PinHeader_1x03_P2.54mm_Vertical, symbol interruptorRev2-rescue:Conn_01x03_Female-RESCUE-termostato-termostato-rescue-in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
- removed Q1, Q2: PN2222A, Package_TO_SOT_SMD:SOT-23, symbol interruptorRev2-rescue:PN2222A-pn2222a
- added Q1, Q2: 2N7002, Package_TO_SOT_SMD:SOT-23, symbol Transistor_FET:2N7002
Connections:
- net int_1 is gone; now on net Relay_1: U3.6 (GPIO12)
- net GND: now also Q1.2 (S), Q2.2 (S)
- net Relay_1: no longer U3.5 (GPIO14)
- net GPIO5: now reaches U3.14 (GPIO5)
- net at D1.1 (K), U4.4 (-): now also Q1.3 (D)
- net at D2.1 (K), U5.4 (-): now also Q2.3 (D)
- net at R4.1: now also Q1.1 (G)
- net at R5.1: now also Q2.1 (G)
- net int_2 renamed GPIO13
- net vcc renamed VCC
- new net GPIO14: U3.5 (GPIO14)
- no-connect marks 5 -> 4
Changed lines of the file:
@@
 $Descr A4 11693 8268
 encoding utf-8
-Sheet 1 1
+Sheet 1 2
 Title ""
 Date ""
@@
 	1    0    0    -1
 $EndComp
-Text GLabel 5750 5250 0    50   Input ~ 0
-Relay_1
 Text GLabel 5500 5150 0    50   Input ~ 0
 Relay_2
@@
 	4300 4000 4300 4150
 Wire Wire Line
-	5750 5250 5900 5250
+	5100 5250 5900 5250
 Wire Wire Line
 	5750 5350 5900 5350
@@
 Wire Wire Line
 	5800 2450 5800 2800
-Text GLabel 5750 5350 0    50   Input ~ 0
-int_1
 Connection ~ 6800 6050
 $Comp
@@
 Wire Wire Line
 	5500 5150 5900 5150
-$Comp
-L interruptorRev2-rescue:Conn_01x03_Female-RESCUE-termostato-termostato-rescue-interruptor-rescue J5
-U 1 1 5CDD1000
-P 4350 6000
-F 0 "J5" H 4350 6200 50  0000 C CNN
-F 1 "Int_1" H 4250 5800 50  0000 C CNN
-F 2 "Connector_PinHeader_2.54mm:PinHeader_1x03_P2.54mm_Vertical" H 4350 6000 50  0001 C CNN
-F 3 "" H 4350 6000 50  0001 C CNN
-	1    4350 6000
-	0    -1   -1   0
-$EndComp
-Text GLabel 4350 6550 3    50   Input ~ 0
-int_1
-Wire Wire Line
-	4350 6550 4350 6200
-$Comp
-L interruptorRev2-rescue:GND-RESCUE-termostato-termostato-rescue-interruptor-rescue #PWR?
-U 1 1 5CDD4154
-P 4450 6300
-F 0 "#PWR?" H 4450 6050 50  0001 C CNN
-F 1 "GND" H 4450 6150 50  0000 C CNN
-F 2 "" H 4450 6300 50  0001 C CNN
-F 3 "" H 4450 6300 50  0001 C CNN
-	1    4450 6300
-	1    0    0    -1
-$EndComp
-Wire Wire Line
-	4450 6300 4450 6200
-Text GLabel 5300 4600 1    50   Input ~ 0
-vcc
 Wire Wire Line
 	5300 4600 5300 4800
 Wire Wire Line
 	5300 4800 5500 4800
-Text GLabel 4250 6350 3    50   Input ~ 0
-vcc
-Wire Wire Line
-	4250 6350 4250 6200
 $Comp
 L interruptorRev2-rescue:GND-RESCUE-termostato-termostato-rescue-interruptor-rescue #PWR?
@@
 Wire Wire Line
 	9100 5250 9250 5250
-$Comp
-L interruptorRev2-rescue:Conn_01x03_Female-RESCUE-termostato-termostato-rescue-interruptor-rescue J6
-U 1 1 5CDD93D9
-P 5100 6000
-F 0 "J6" H 5100 6200 50  0000 C CNN
-F 1 "int_2" H 5000 5800 50  0000 C CNN
-F 2 "Connector_PinHeader_2.54mm:PinHeader_1x03_P2.54mm_Vertical" H 5100 6000 50  0001 C CNN
-F 3 "" H 5100 6000 50  0001 C CNN
-	1    5100 6000
-	0    -1   -1   0
-$EndComp
-Text GLabel 5100 6550 3    50   Input ~ 0
-int_2
-Wire Wire Line
-	5100 6550 5100 6200
-$Comp
-L interruptorRev2-rescue:GND-RESCUE-termostato-termostato-rescue-interruptor-rescue #PWR?
-U 1 1 5CDD93E1
-P 5200 6300
-F 0 "#PWR?" H 5200 6050 50  0001 C CNN
-F 1 "GND" H 5200 6150 50  0000 C CNN
-F 2 "" H 5200 6300 50  0001 C CNN
-F 3 "" H 5200 6300 50  0001 C CNN
-	1    5200 6300
-	1    0    0    -1
-$EndComp
-Wire Wire Line
-	5200 6300 5200 6200
-Text GLabel 5000 6350 3    50   Input ~ 0
-vcc
-Wire Wire Line
-	5000 6350 5000 6200
-Text GLabel 5650 5450 0    50   Input ~ 0
-int_2
-Wire Wire Line
-	5650 5450 5900 5450
+Wire Wire Line
+	5100 5450 5900 5450
 Wire Wire Line
 	7700 5250 9000 5250
 Wire Wire Line
 	2500 4750 2750 4750
-$Comp
-L interruptorRev2-rescue:PN2222A-pn2222a Q1
-U 1 1 5CEFE5BD
-P 4500 3150
-F 0 "Q1" H 4691 3196 50  0000 L CNN
-F 1 "PN2222A" H 4691 3105 50  0000 L CNN
-F 2 "Package_TO_SOT_SMD:SOT-23" H 4700 3075 50  0001 L CIN
-F 3 "http://www.fairchildsemi.com/ds/PN/PN2222A.pdf" H 4500 3150 50  0001 L CNN
-	1    4500 3150
-	1    0    0    -1
-$EndComp
-$Comp
-L interruptorRev2-rescue:PN2222A-pn2222a Q2
-U 1 1 5CEFE632
-P 6000 3150
-F 0 "Q2" H 6191 3196 50  0000 L CNN
-F 1 "PN2222A" H 6191 3105 50  0000 L CNN
-F 2 "Package_TO_SOT_SMD:SOT-23" H 6200 3075 50  0001 L CIN
-F 3 "http://www.fairchildsemi.com/ds/PN/PN2222A.pdf" H 6000 3150 50  0001 L CNN
-	1    6000 3150
-	1    0    0    -1
-$EndComp
-NoConn ~ 7700 5050
 $Comp
 L interruptorRev2-rescue:JRC-21(4100)-reles U4
@@
 	5150 1800 5150 2450
 Text GLabel 3950 4750 2    50   Input ~ 0
-vcc
+VCC
 $Comp
 L Connector_Generic:Conn_01x04 J2
@@
 	0    -1   -1   0
 $EndComp
+$Sheet
+S 8150 850  2000 1050
+U 5D5B915E
+F0 "Sheet5D5B915D" 50
+F1 "file5D5B915D.sch" 50
+$EndSheet
+$Comp
+L Transistor_FET:2N7002 Q1
+U 1 1 5D5D3125
+P 4500 3150
+F 0 "Q1" H 4705 3196 50  0000 L CNN
+F 1 "2N7002" H 4705 3105 50  0000 L CNN
+F 2 "Package_TO_SOT_SMD:SOT-23" H 4700 3075 50  0001 L CIN
+F 3 "https://www.fairchildsemi.com/datasheets/2N/2N7002.pdf" H 4500 3150 50  0001 L CNN
+	1    4500 3150
+	1    0    0    -1
+$EndComp
+$Comp
+L Transistor_FET:2N7002 Q2
+U 1 1 5D5D31D0
+P 6000 3150
+F 0 "Q2" H 6205 3196 50  0000 L CNN
+F 1 "2N7002" H 6205 3105 50  0000 L CNN
+F 2 "Package_TO_SOT_SMD:SOT-23" H 6200 3075 50  0001 L CIN
+F 3 "https://www.fairchildsemi.com/datasheets/2N/2N7002.pdf" H 6000 3150 50  0001 L CNN
+	1    6000 3150
+	1    0    0    -1
+$EndComp
+Text GLabel 5750 5350 0    50   Input ~ 0
+Relay_1
+Text GLabel 5100 5250 0    50   Input ~ 0
+GPIO14
+Text GLabel 5100 5450 0    50   Input ~ 0
+GPIO13
+Wire Wire Line
+	7700 5050 8150 5050
+Text GLabel 8150 5050 2    50   Input ~ 0
+GPIO5
+Text GLabel 5300 4600 1    50   Input ~ 0
+VCC
 $EndSCHEMATC

Commit message: esquema dividido por secciones
Parts:
- removed D1, D2: DIODE, Diode_SMD:D_1206_3216Metric_Pad1.42x1.75mm_HandSolder, symbol pspice:DIODE
- removed J1: 220v, TerminalBlock:TerminalBlock_bornier-2_P5.08mm, symbol interruptorRev2-rescue:Conn_01x02_Female-RESCUE-termostato-termostato-rescue-in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
- removed J3, J4: Screw_Terminal_01x03, TerminalBlock:TerminalBlock_bornier-3_P5.08mm, symbol Connector:Screw_Terminal_01x03
- added D1, D2: 1N4148, espurna-h:SOD80, symbol Diode:1N4148
- added J1, J3, J4: Screw_Terminal_01x02, symbol Connector:Screw_Terminal_01x02
- R1, R2, R3, R4, R5: footprint Resistor_SMD:R_1206_3216Metric_Pad1.42x1.75mm_HandSolder -> Resistor_SMD:R_0805_2012Metric_Pad1.15x1.40mm_HandSolder
Connections:
- net VCC: now also D1.1 (K), D2.1 (K)
- net NEUTRAL: now reaches U1.P$2 (AC2)
- net NEUTRAL: now also J1.1 (Pin_1)
- net LINE_I: now reaches U1.P$1 (AC1)
- net LINE_I: now also J1.2 (Pin_2)
- net at Q1.3 (D), U4.4 (-): now also D1.2 (A)
- net at Q2.3 (D), U5.4 (-): now also D2.2 (A)
- net at U4.5 (nc): now also J3.1 (Pin_1)
- net at U4.2 (L): no longer U4.1 (L)
- net at U4.6 (no): now also J3.2 (Pin_2)
- net at U5.5 (nc): now also J4.1 (Pin_1)
- net at U5.1 (L): no longer U5.2 (L)
- net at U5.6 (no): now also J4.2 (Pin_2)
- new net LINE_L: U4.1 (L)
- no-connect marks 4 -> 7
Changed lines of the file:
@@
 Comment4 ""
 $EndDescr
-$Comp
-L interruptorRev2-rescue:Conn_01x02_Female-RESCUE-termostato-termostato-rescue-interruptor-rescue J1
-U 1 1 5A3E8B13
-P 2300 5000
-F 0 "J1" H 2300 5100 50  0000 C CNN
-F 1 "220v" H 2300 4800 50  0000 C CNN
-F 2 "TerminalBlock:TerminalBlock_bornier-2_P5.08mm" H 2300 5000 50  0001 C CNN
-F 3 "" H 2300 5000 50  0001 C CNN
-	1    2300 5000
-	-1   0    0    1
-$EndComp
 NoConn ~ 5900 4850
 NoConn ~ 5900 4950
@@
 F 0 "R3" V 7880 4650 50  0000 C CNN
 F 1 "180" V 7800 4650 50  0000 C CNN
-F 2 "Resistor_SMD:R_1206_3216Metric_Pad1.42x1.75mm_HandSolder" V 7730 4650 50  0001 C CNN
+F 2 "Resistor_SMD:R_0805_2012Metric_Pad1.15x1.40mm_HandSolder" V 7730 4650 50  0001 C CNN
 F 3 "" H 7800 4650 50  0001 C CNN
 	1    7800 4650
@@
 F 0 "R2" V 7780 5750 50  0000 C CNN
 F 1 "10K" V 7700 5750 50  0000 C CNN
-F 2 "Resistor_SMD:R_1206_3216Metric_Pad1.42x1.75mm_HandSolder" V 7630 5750 50  0001 C CNN
+F 2 "Resistor_SMD:R_0805_2012Metric_Pad1.15x1.40mm_HandSolder" V 7630 5750 50  0001 C CNN
 F 3 "" H 7700 5750 50  0001 C CNN
 	1    7700 5750
@@
 F 0 "R1" V 5780 5050 50  0000 C CNN
 F 1 "10K" V 5700 5050 50  0000 C CNN
-F 2 "Resistor_SMD:R_1206_3216Metric_Pad1.42x1.75mm_HandSolder" V 5630 5050 50  0001 C CNN
+F 2 "Resistor_SMD:R_0805_2012Metric_Pad1.15x1.40mm_HandSolder" V 5630 5050 50  0001 C CNN
 F 3 "" H 5700 5050 50  0001 C CNN
 	1    5700 5050
@@
 $EndComp
 Wire Wire Line
-	2500 4900 2500 4750
-Wire Wire Line
-	2500 5000 2500 5150
-Wire Wire Line
-	2500 5150 2750 5150
+	2350 5150 2750 5150
 Wire Wire Line
 	3750 5150 3750 5300
@@
 	1    0    0    -1
 $EndComp
-$Comp
-L pspice:DIODE D1
-U 1 1 5CD2F6F3
-P 4150 2150
-F 0 "D1" H 4150 2000 50  0000 C CNN
-F 1 "DIODE" H 4150 2300 50  0000 C CNN
-F 2 "Diode_SMD:D_1206_3216Metric_Pad1.42x1.75mm_HandSolder" H 4150 2150 50  0001 C CNN
-F 3 "~" H 4150 2150 50  0001 C CNN
-	1    4150 2150
-	-1   0    0    1
-$EndComp
-$Comp
-L pspice:DIODE D2
-U 1 1 5CD326D9
-P 5600 2450
-F 0 "D2" H 5600 2185 50  0000 C CNN
-F 1 "DIODE" H 5600 2276 50  0000 C CNN
-F 2 "Diode_SMD:D_1206_3216Metric_Pad1.42x1.75mm_HandSolder" H 5600 2450 50  0001 C CNN
-F 3 "~" H 5600 2450 50  0001 C CNN
-	1    5600 2450
-	-1   0    0    1
-$EndComp
 Wire Wire Line
 	3750 2550 5400 2550
@@
 	5400 2550 5400 2450
 Connection ~ 3750 2550
-Wire Wire Line
-	4350 2150 4400 2150
 $Comp
 L Device:R R4
@@
 F 0 "R4" H 4370 3896 50  0000 L CNN
 F 1 "180" H 4370 3805 50  0000 L CNN
-F 2 "Resistor_SMD:R_1206_3216Metric_Pad1.42x1.75mm_HandSolder" V 4230 3850 50  0001 C CNN
+F 2 "Resistor_SMD:R_0805_2012Metric_Pad1.15x1.40mm_HandSolder" V 4230 3850 50  0001 C CNN
 F 3 "~" H 4300 3850 50  0001 C CNN
 	1    4300 3850
@@
 F 0 "R5" H 5870 3896 50  0000 L CNN
 F 1 "180" H 5870 3805 50  0000 L CNN
-F 2 "Resistor_SMD:R_1206_3216Metric_Pad1.42x1.75mm_HandSolder" V 5730 3850 50  0001 C CNN
+F 2 "Resistor_SMD:R_0805_2012Metric_Pad1.15x1.40mm_HandSolder" V 5730 3850 50  0001 C CNN
 F 3 "~" H 5800 3850 50  0001 C CNN
 	1    5800 3850
@@
 Wire Wire Line
 	3750 4750 3950 4750
-$Comp
-L Connector:Screw_Terminal_01x03 J3
-U 1 1 5CD5F5C6
-P 4150 900
-F 0 "J3" V 4116 712 50  0000 R CNN
-F 1 "Screw_Terminal_01x03" V 4025 712 50  0000 R CNN
-F 2 "TerminalBlock:TerminalBlock_bornier-3_P5.08mm" H 4150 900 50  0001 C CNN
-F 3 "~" H 4150 900 50  0001 C CNN
-	1    4150 900
-	0    -1   -1   0
-$EndComp
-$Comp
-L Connector:Screw_Terminal_01x03 J4
-U 1 1 5CD62DF4
-P 5550 900
-F 0 "J4" V 5516 712 50  0000 R CNN
-F 1 "Screw_Terminal_01x03" V 5425 712 50  0000 R CNN
-F 2 "TerminalBlock:TerminalBlock_bornier-3_P5.08mm" H 5550 900 50  0001 C CNN
-F 3 "~" H 5550 900 50  0001 C CNN
-	1    5550 900
-	0    -1   -1   0
-$EndComp
 Wire Wire Line
 	7000 4100 7000 4500
@@
 	7700 5250 9000 5250
 Wire Wire Line
-	2500 4750 2750 4750
+	2350 4750 2750 4750
 $Comp
 L interruptorRev2-rescue:JRC-21(4100)-reles U4
@@
 Wire Wire Line
 	4500 1750 4500 2150
-Connection ~ 4400 2150
 Wire Wire Line
 	4600 1100 4600 1850
@@
 	4600 1850 4400 1850
 Wire Wire Line
-	4250 1100 4600 1100
+	4150 1100 4600 1100
 Wire Wire Line
 	3700 1100 3700 1850
@@
 Wire Wire Line
 	3700 1100 4050 1100
-Wire Wire Line
-	4150 1100 4150 1200
-Wire Wire Line
-	4150 1200 4400 1200
-Wire Wire Line
-	4400 1200 4400 1450
-Wire Wire Line
-	4150 1200 3850 1200
-Wire Wire Line
-	3850 1200 3850 1450
-Connection ~ 4150 1200
 $Comp
 L interruptorRev2-rescue:JRC-21(4100)-reles U5
@@
 Wire Wire Line
 	5150 2450 5400 2450
-Connection ~ 5400 2450
 Wire Wire Line
 	5850 1800 5950 1800
@@
 Wire Wire Line
 	5950 2450 5800 2450
-Connection ~ 5800 2450
 Wire Wire Line
 	5450 1100 5250 1100
@@
 	5250 1900 5300 1900
 Wire Wire Line
-	5650 1100 5900 1100
+	5550 1100 5900 1100
 Wire Wire Line
 	5900 1100 5900 1900
 Wire Wire Line
 	5900 1900 5850 1900
-Wire Wire Line
-	5300 1500 5300 1200
-Wire Wire Line
-	5300 1200 5550 1200
-Wire Wire Line
-	5550 1200 5550 1100
-Wire Wire Line
-	5850 1500 5850 1200
-Wire Wire Line
-	5850 1200 5550 1200
-Connection ~ 5550 1200
 Wire Wire Line
 	3750 2550 3750 4750
@@
 $EndComp
 $Sheet
-S 8150 850  2000 1050
+S 12600 100  2000 1050
 U 5D5B915E
 F0 "Sheet5D5B915D" 50
@@
 Text GLabel 5300 4600 1    50   Input ~ 0
 VCC
+$Comp
+L Diode:1N4148 D1
+U 1 1 5D5C40DC
+P 4100 2150
+F 0 "D1" H 4100 2366 50  0000 C CNN
+F 1 "1N4148" H 4100 2275 50  0000 C CNN
+F 2 "espurna-h:SOD80" H 4100 1975 50  0001 C CNN
+F 3 "http://www.nxp.com/documents/data_sheet/1N4148_1N4448.pdf" H 4100 2150 50  0001 C CNN
+	1    4100 2150
+	1    0    0    -1
+$EndComp
+Wire Wire Line
+	4250 2150 4400 2150
+Connection ~ 4400 2150
+$Comp
+L Diode:1N4148 D2
+U 1 1 5D5C9A7E
+P 5600 2450
+F 0 "D2" H 5600 2666 50  0000 C CNN
+F 1 "1N4148" H 5600 2575 50  0000 C CNN
+F 2 "espurna-h:SOD80" H 5600 2275 50  0001 C CNN
+F 3 "http://www.nxp.com/documents/data_sheet/1N4148_1N4448.pdf" H 5600 2450 50  0001 C CNN
+	1    5600 2450
+	1    0    0    -1
+$EndComp
+Wire Wire Line
+	5400 2450 5450 2450
+Connection ~ 5400 2450
+Wire Wire Line
+	5750 2450 5800 2450
+Connection ~ 5800 2450
+Text GLabel 1650 4200 2    50   Input ~ 0
+NEUTRAL
+Text GLabel 2350 5150 0    50   Input ~ 0
+NEUTRAL
+Text GLabel 1650 4100 2    50   Input ~ 0
+LINE_I
+Text GLabel 2350 4750 0    50   Input ~ 0
+LINE_I
+$Comp
+L Connector:Screw_Terminal_01x02 J1
+U 1 1 5D5EA3D7
+P 1450 4200
+F 0 "J1" H 1370 3875 50  0000 C CNN
+F 1 "Screw_Terminal_01x02" H 1370 3966 50  0000 C CNN
+F 2 "" H 1450 4200 50  0001 C CNN
+F 3 "~" H 1450 4200 50  0001 C CNN
+	1    1450 4200
+	-1   0    0    1
+$EndComp
+$Comp
+L Connector:Screw_Terminal_01x02 J3
+U 1 1 5D5EA93C
+P 4050 900
+F 0 "J3" V 4016 712 50  0000 R CNN
+F 1 "Screw_Terminal_01x02" V 3925 712 50  0000 R CNN
+F 2 "" H 4050 900 50  0001 C CNN
+F 3 "~" H 4050 900 50  0001 C CNN
+	1    4050 900
+	0    -1   -1   0
+$EndComp
+$Comp
+L Connector:Screw_Terminal_01x02 J4
+U 1 1 5D5ECB90
+P 5450 900
+F 0 "J4" V 5416 712 50  0000 R CNN
+F 1 "Screw_Terminal_01x02" V 5325 712 50  0000 R CNN
+F 2 "" H 5450 900 50  0001 C CNN
+F 3 "~" H 5450 900 50  0001 C CNN
+	1    5450 900
+	0    -1   -1   0
+$EndComp
+Wire Wire Line
+	3850 1450 3350 1450
+Text GLabel 3350 1450 0    50   Input ~ 0
+LINE_L
+NoConn ~ 4400 1450
+NoConn ~ 5300 1500
+NoConn ~ 5850 1500
 $EndSCHEMATC
